File: Electronics/botctrl-rev2/botctrl.kicad_sch (KiCad schematic)
At the start: 72 parts, among them J1 Conn_02x01, J12 Conn_01x03_Pin, J13 Conn_01x01_Pin, J14 Conn_01x01_Pin, J2 Conn_02x01, J3 Conn_01x03_Pin, U1 ADS1115IDGS, U13 LDL212PU50R, U3 MPU-6050, U4 MOUDLE-SEEEDUINO-XIAO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

Commit message: updated to latest version
Other:
- note added: "DRIVE"
- note added: "IMU"
- note added: "POWER INPUT"
- note added: "RGB"
- moved on the sheet: C2, D13, D8, FID1, H1, J12, J3, R10, R12, R22, R25, U1
