File: Electronics/botctrl-rev2/drive.kicad_sch (KiCad schematic)
At the start: 21 parts, among them J10 Conn_01x01_Pin, J11 Conn_01x01_Pin, U10 DRV8256PRGER

Commit message: updated to latest version
Parts:
- renumbered C56 to C10, C55 to C19, C30 to C20, C58 to C22, C59 to C23, C61 to C25, C62 to C26, C63 to C27, C65 to C29, C40 to C32, C71 to C68, C75 to C72, D12 to D9, J10 to J4, J11 to J5, R21 to R11, R44 to R14, R48 to R18, R49 to R19, R16 to R9, U10 to U7
Changed lines of the file:
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@@
 (kicad_sch
-	(version 20231120)
+	(version 20250114)
 	(generator "eeschema")
-	(generator_version "8.0")
+	(generator_version "9.0")
 	(paper "A4")
 	(junction
@@
 		(on_board yes)
 		(dnp no)
-		(property "Reference" "C30"
+		(property "Reference" "C20"
 			(at 143.51 55.8736 0)
 			(effects
@@
 		(dnp no)
 		(fields_autoplaced yes)
-		(property "Reference" "C58"
+		(property "Reference" "C22"
 			(at 166.37 55.8862 0)
 			(effects
@@
 		(dnp no)
 		(fields_autoplaced yes)
-		(property "Reference" "C61"
+		(property "Reference" "C25"
 			(at 180.3463 80.01 90)
 			(effects
@@
 		(on_board yes)
 		(dnp no)
-		(property "Reference" "R44"
+		(property "Reference" "R14"
 			(at 125.73 90.1699 0)
 			(effects
@@
 		(on_board yes)
 		(dnp no)
-		(property "Reference" "C75"
+		(property "Reference" "C72"
 			(at 209.55 106.6735 0)
 			(effects
@@
 		(dnp no)
 		(fields_autoplaced yes)
-		(property "Reference" "D12"
+		(property "Reference" "D9"
 			(at 107.95 90.17 0)
 			(effects
@@
 		(on_board yes)
 		(dnp no)
-		(property "Reference" "C71"
+		(property "Reference" "C68"
 			(at 200.66 106.6735 0)
 			(effects
@@
 		(dnp no)
 		(fields_autoplaced yes)
-		(property "Reference" "#PWR051"
+		(property "Reference" "#PWR047"
 			(at 205.74 119.38 0)
 			(effects
@@
 		(dnp no)
 		(fields_autoplaced yes)
-		(property "Reference" "C59"
+		(property "Reference" "C23"
 			(at 173.99 55.8862 0)
 			(effects
@@
 		(on_board yes)
 		(dnp no)
-		(property "Reference" "R48"
+		(property "Reference" "R18"
 			(at 128.27 118.1099 0)
 			(effects
@@
 		(dnp no)
 		(fields_autoplaced yes)
-		(property "Reference" "R21"
+		(property "Reference" "R11"
 			(at 196.85 114.3 90)
 			(effects
@@
 		(dnp no)
 		(fields_autoplaced yes)
-		(property "Reference" "#PWR048"
+		(property "Reference" "#PWR039"
 			(at 187.96 140.97 0)
 			(effects
@@
 		(on_board yes)
 		(dnp no)
-		(property "Reference" "C65"
+		(property "Reference" "C29"
 			(at 209.55 100.3235 0)
 			(effects
@@
 		(dnp no)
 		(fields_autoplaced yes)
-		(property "Reference" "R16"
+		(property "Reference" "R9"
 			(at 81.28 100.33 90)
 			(effects
@@
 		(dnp no)
 		(fields_autoplaced yes)
-		(property "Reference" "#PWR038"
+		(property "Reference" "#PWR015"
 			(at 154.94 68.58 0)
 			(effects
@@
 		(on_board yes)
 		(dnp no)
-		(property "Reference" "C40"
+		(property "Reference" "C32"
 			(at 152.4 55.8736 0)
 			(effects
@@
 		(dnp no)
 		(fields_autoplaced yes)
-		(property "Reference" "U10"
+		(property "Reference" "U7"
 			(at 157.48 73.66 0)
 			(effects
@@
 		(dnp no)
 		(fields_autoplaced yes)
-		(property "Reference" "J10"
+		(property "Reference" "J4"
 			(at 222.885 93.98 0)
 			(effects
@@
 		(dnp no)
 		(fields_autoplaced yes)
-		(property "Reference" "C62"
+		(property "Reference" "C26"
 			(at 190.5 85.0962 0)
 			(effects
@@
 		(on_board yes)
 		(dnp no)
-		(property "Reference" "J11"
+		(property "Reference" "J5"
 			(at 222.885 109.22 0)
 			(effects
@@
 		(on_board yes)
 		(dnp no)
-		(property "Reference" "C63"
+		(property "Reference" "C27"
 			(at 204.47 124.4662 0)
 			(effects
@@
 		(on_board yes)
 		(dnp no)
-		(property "Reference" "C55"
+		(property "Reference" "C19"
 			(at 137.16 96.5262 0)
 			(effects
@@
 		(on_board yes)
 		(dnp no)
-		(property "Reference" "C56"
+		(property "Reference" "C10"
 			(at 90.17 109.2262 0)
 			(effects
@@
 		(dnp no)
 		(fields_autoplaced yes)
-		(property "Reference" "R49"
+		(property "Reference" "R19"
 			(at 190.5 123.1899 0)
 			(effects
